Commit message: Integrating excel_description with new UR10 model.
The files ur10_new... have been integrated into the
new ur_description, so a copy is no longer needed here.

File: excel_description/urdf/excel_robot.urdf.xacro (robot description, xacro)
@@ -4,12 +4,9 @@
   Contributers: Kelsey Hawkins, Ajit Krisshna N L, Muhammad Asif Rana
 -->
-<robot xmlns:controller="http://playerstage.sourceforge.net/gazebo/xmlschema/#controller"
-	xmlns:interface="http://playerstage.sourceforge.net/gazebo/xmlschema/#interface"
-	xmlns:sensor="http://playerstage.sourceforge.net/gazebo/xmlschema/#sensor"
-	xmlns:xacro="http://playerstage.sourceforge.net/gazebo/xmlschema/#interface" name="excel">
+<robot xmlns:xacro="http://playerstage.sourceforge.net/gazebo/xmlschema/#interface" name="excel">
    <!-- common stuff -->
    <xacro:include filename="$(find ur_description)/urdf/gazebo.urdf.xacro" />
    <!-- include ur10 -->
-   <xacro:include filename="$(find excel_description)/urdf/ur10_new.urdf.xacro" />
+   <xacro:include filename="$(find ur_description)/urdf/ur10.urdf.xacro" />
    <!-- include table&rail -->
    <xacro:include filename="$(find excel_description)/urdf/table_rail.urdf.xacro" />

File: excel_description/urdf/table_rail.gazebo.xacro (robot description, xacro)
@@ -4,8 +4,5 @@
   Contributers: Kelsey Hawkins, Ajit Krisshna N L, Muhammad Asif Rana
 -->
-<robot xmlns:controller="http://playerstage.sourceforge.net/gazebo/xmlschema/#controller"
-	xmlns:interface="http://playerstage.sourceforge.net/gazebo/xmlschema/#interface"
-	xmlns:sensor="http://playerstage.sourceforge.net/gazebo/xmlschema/#sensor"
-	xmlns:xacro="http://ros.org/wiki/xacro">
+<robot xmlns:xacro="http://ros.org/wiki/xacro">
    <xacro:macro name="table_rail_gazebo" params="prefix">
       <gazebo reference="${prefix}table_link">

File: excel_description/urdf/table_rail.transmission.xacro (robot description, xacro)
@@ -4,8 +4,5 @@
   Contributers: Kelsey Hawkins, Ajit Krisshna N L, Muhammad Asif Rana
 -->
-<robot xmlns:controller="http://playerstage.sourceforge.net/gazebo/xmlschema/#controller"
-	xmlns:interface="http://playerstage.sourceforge.net/gazebo/xmlschema/#interface"
-	xmlns:sensor="http://playerstage.sourceforge.net/gazebo/xmlschema/#sensor"
-	xmlns:xacro="http://ros.org/wiki/xacro">
+<robot xmlns:xacro="http://ros.org/wiki/xacro">
    <xacro:macro name="table_rail_transmission" params="prefix">
       <transmission name="rail_base_trans" type="pr2_mechanism_model/SimpleTransmission">

File: excel_description/urdf/table_rail.urdf.xacro (robot description, xacro)
@@ -4,8 +4,5 @@
   Contributers: Kelsey Hawkins, Ajit Krisshna N L, Muhammad Asif Rana
 -->
-<robot xmlns:controller="http://playerstage.sourceforge.net/gazebo/xmlschema/#controller"
-	xmlns:interface="http://playerstage.sourceforge.net/gazebo/xmlschema/#interface"
-	xmlns:sensor="http://playerstage.sourceforge.net/gazebo/xmlschema/#sensor"
-	xmlns:xacro="http://ros.org/wiki/xacro">
+<robot xmlns:xacro="http://ros.org/wiki/xacro">
    <xacro:include filename="$(find excel_description)/urdf/table_rail.transmission.xacro" />
    <xacro:include filename="$(find excel_description)/urdf/table_rail.gazebo.xacro" />
@@ -34,8 +31,11 @@
          </collision>
       </link>
-      <joint name="${prefix}table_rail_joint" type="fixed">
+      <joint name="${prefix}table_rail_joint" type="prismatic">
          <parent link="${prefix}table_link" />
          <child link="${prefix}rail_link" />
          <origin rpy="0.0 0.0 0.0" xyz="${table_collision_offset}" />
+         <axis xyz="0 1 0" />
+         <limit effort="10.0" lower="0.0" upper="${rail_length}" velocity="${pi}" />
+         <dynamics damping="10" friction="0.1" />
       </joint>
       <link name="${prefix}rail_link">
@@ -45,11 +45,8 @@
          </inertial>
       </link>
-      <joint name="${prefix}rail_base_joint" type="prismatic">
+      <joint name="${prefix}rail_base_joint" type="fixed">
          <parent link="${prefix}rail_link" />
          <child link="${prefix}base_link" />
          <origin rpy="0.0 0.0 0.0" xyz="0.0 0.0 0.0" />
-         <axis xyz="0 1 0" />
-         <limit effort="10.0" lower="0.0" upper="${rail_length}" velocity="${pi}" />
-         <dynamics damping="10" friction="0.1" />
       </joint>
       <xacro:table_rail_transmission prefix="${prefix}" />

Commit message: Excel jogging control fully working

File: excel_description/urdf/excel_robot.urdf.xacro (robot description, xacro)
@@ -8,5 +8,5 @@
    <xacro:include filename="$(find ur_description)/urdf/gazebo.urdf.xacro" />
    <!-- include ur10 -->
-   <xacro:include filename="$(find excel_description)/urdf/ur10.urdf.xacro" />
+   <xacro:include filename="$(find ur_description)/urdf/ur10.urdf.xacro" />
    <!-- include table&rail -->
    <xacro:include filename="$(find excel_description)/urdf/table_rail.urdf.xacro" />
@@ -14,5 +14,5 @@
    <xacro:include filename="$(find excel_description)/urdf/gripper.urdf.xacro" />
    <!-- ur10 -->
-  <xacro:ur10_robot prefix="" joint_limited="true"/>
+  <xacro:ur10_robot prefix="" joint_limited="false"/>
    <!-- table&rail -->
    <xacro:table_rail prefix="" />

File: excel_description/urdf/table_rail.urdf.xacro (robot description, xacro)
@@ -13,5 +13,6 @@
    <property name="rail_mass" value="50.0" />
    <!-- Kinematic model -->
-   <property name="rail_length" value="3.75" />
+   <property name="rail_lower_limit" value="0.05" />
+   <property name="rail_upper_limit" value="3.45" />
    <!-- Collision model -->
    <property name="table_collision_offset" value="0.80137 0.05588 0.9" />
@@ -36,5 +37,5 @@
          <origin rpy="0.0 0.0 0.0" xyz="${table_collision_offset}" />
          <axis xyz="0 1 0" />
-         <limit effort="10.0" lower="0.0" upper="${rail_length}" velocity="${pi}" />
+         <limit effort="10.0" lower="${rail_lower_limit}" upper="${rail_upper_limit}" velocity="${pi}" />
          <dynamics damping="10" friction="0.1" />
       </joint>
@@ -48,5 +49,5 @@
          <parent link="${prefix}rail_link" />
          <child link="${prefix}base_link" />
-         <origin rpy="0.0 0.0 0.0" xyz="0.0 0.0 0.0" />
+         <origin rpy="0.0 0.0 ${-pi/2}" xyz="0.0 0.0 0.0" />
       </joint>
       <xacro:table_rail_transmission prefix="${prefix}" />
