Commit message: Fixing frame offset error for kinect_frames

File: excel_description/urdf/kinect_frames.urdf.xacro (robot description, xacro)
@@ -24,5 +24,5 @@
     </link>
     <joint name="${camera}_depth_optical_frame_joint" type="fixed">
-      <parent link="${camera}_link" />
+      <parent link="${camera}_depth_frame" />
       <child link="${camera}_depth_optical_frame" />
       <origin xyz="0 0 0" rpy="${optical_rotate}" />
@@ -31,5 +31,5 @@
     </link>
     <joint name="${camera}_rgb_optical_frame_joint" type="fixed">
-      <parent link="${camera}_link" />
+      <parent link="${camera}_rgb_frame" />
       <child link="${camera}_rgb_optical_frame" />
       <origin xyz="0 0 0" rpy="${optical_rotate}" />
