Commit message: Optimizing planning.  Changing default controller to vel/pva

File: excel_description/urdf/excel_robot_moplan.urdf.xacro (robot description, xacro)
@@ -16,5 +16,5 @@
    <xacro:include filename="$(find excel_description)/urdf/cameras.urdf.xacro" />
    <!-- ur10 -->
-  <xacro:ur10_robot prefix="" cylinders_collision="false"
+  <xacro:ur10_robot prefix="" cylinders_collision="true"
                     j1_lwr_lmt="${-2.0*pi}" j1_upr_lmt="${2.0*pi}" j1_vel_lmt="2.16"
                     j2_lwr_lmt="${-pi}" j2_upr_lmt="${0.0}" j2_vel_lmt="2.16"

File: excel_description/urdf/gripper.urdf.xacro (robot description, xacro)
@@ -52,4 +52,16 @@
             <origin rpy="${pi} 0 ${pi / 2.0}" xyz="0 0 0" />
          </visual>
+         <collision>
+            <geometry>
+              <box size="0.03 0.16 0.055" />
+            </geometry>
+            <origin xyz="0.015 -0.01 0.005" rpy="0 0 0" />
+         </collision>
+         <collision>
+            <geometry>
+              <box size="0.045 0.05 0.038" />
+            </geometry>
+            <origin xyz="0.053 0.0 -0.01" rpy="0 0 0" />
+         </collision>
       </link>
       <joint name="${prefix}robotiq_85_left_knuckle_joint" type="fixed">
@@ -196,4 +208,10 @@
             <origin rpy="0 ${pi/2.0} 0" xyz="0 -.090381 .051505" />
          </visual>
+         <collision>
+            <geometry>
+              <box size="0.038 0.12 0.05" />
+            </geometry>
+            <origin xyz="0.01 0.00 0" rpy="0 0 0" />
+         </collision>
       </link>
       <joint name="${prefix}robotiq_85_right_finger_tip_joint" type="fixed">
@@ -217,4 +235,10 @@
             <origin rpy="0 ${-pi/2.0} 0" xyz="0 -.090381 .051505" />
          </visual>
+         <collision>
+            <geometry>
+              <box size="0.038 0.12 0.05" />
+            </geometry>
+            <origin xyz="-0.01 0.00 0" rpy="0 0 0" />
+         </collision>
       </link>
    </xacro:macro>

File: excel_description/urdf/table_rail.urdf.xacro (robot description, xacro)
@@ -25,7 +25,31 @@
          <collision>
             <geometry>
-               <mesh filename="package://excel_description/meshes/collision/tables+rail.stl"/>
+              <box size="0.92 2.25 0.87" />
             </geometry>
-            <origin rpy="0.0 0.0 0.0" xyz="0.0 0.0 0.0" />
+            <origin xyz="0.46 1.125 0.435" rpy="0 0 0" />
+         </collision>
+         <collision>
+            <geometry>
+              <box size="3.97 0.92 0.87" />
+            </geometry>
+            <origin xyz="1.985 0.46 0.435" rpy="0 0 0" />
+         </collision>
+         <collision>
+            <geometry>
+              <box size="0.92 2.0 0.87" />
+            </geometry>
+            <origin xyz="3.5 1.0 0.435" rpy="0 0 0" />
+         </collision>
+         <collision>
+            <geometry>
+              <box size="0.92 0.64 1.34" />
+            </geometry>
+            <origin xyz="3.5 -0.04 0.67" rpy="0 0 0" />
+         </collision>
+         <collision>
+            <geometry>
+              <box size="3.9 0.124 0.065" />
+            </geometry>
+            <origin xyz="1.847 0.811 0.905" rpy="0 0 0" />
          </collision>
       </link>
