Commit message: Simplifying the collision file for the table+rail

File: excel_description/urdf/table_rail.urdf.xacro (robot description, xacro)
@@ -26,5 +26,5 @@
          <collision>
             <geometry>
-               <mesh filename="package://excel_description/meshes/collision/table_collision.stl" />
+               <mesh filename="package://excel_description/meshes/collision/table+rail_collision.stl" />
             </geometry>
             <origin rpy="0.0 0.0 0.0" xyz="0 0.0 0" />

Commit message: Modifying the urdf to match with the actual world

File: excel_description/urdf/table_rail.urdf.xacro (robot description, xacro)
@@ -13,20 +13,20 @@
    <property name="rail_mass" value="50.0" />
    <!-- Kinematic model -->
-   <property name="rail_length" value="3.75" />
+   <property name="rail_length" value="3.54" />
    <!-- Collision model -->
-   <property name="table_collision_offset" value="0.80137 0.05588 0.9" />
+   <property name="table_collision_offset" value="0.135 0.81 0.935" />
    <xacro:macro name="table_rail" params="prefix">
       <link name="${prefix}table_link">
          <visual>
             <geometry>
-               <mesh filename="package://excel_description/meshes/visual/table+rail.dae" />
+               <mesh filename="package://excel_description/meshes/visual/tables+rail.dae"/>
             </geometry>
-            <origin rpy="0.0 0.0 0.0" xyz="0 0.0 0" />
+            <origin rpy="0.0 0.0 0.0" xyz="0.0 0.0 0.0" />
          </visual>
          <collision>
             <geometry>
-               <mesh filename="package://excel_description/meshes/collision/table+rail_collision.stl" />
+               <mesh filename="package://excel_description/meshes/collision/tables+rail.stl"/>
             </geometry>
-            <origin rpy="0.0 0.0 0.0" xyz="0 0.0 0" />
+            <origin rpy="0.0 0.0 0.0" xyz="0.0 0.0 0.0" />
          </collision>
       </link>
@@ -35,5 +35,5 @@
          <child link="${prefix}rail_link" />
          <origin rpy="0.0 0.0 0.0" xyz="${table_collision_offset}" />
-         <axis xyz="0 1 0" />
+         <axis xyz="1 0 0" />
          <limit effort="10.0" lower="0.0" upper="${rail_length}" velocity="${pi}" />
          <dynamics damping="10" friction="0.1" />

File: excel_description/urdf/ur10.urdf.xacro (robot description, xacro)
@@ -145,5 +145,5 @@
       </xacro:unless>
       <xacro:if value="${joint_limited}">
-        <limit lower="${-pi}" upper="${0}" effort="150.0" velocity="3.15"/>
+        <limit lower="${0}" upper="${pi}" effort="150.0" velocity="3.15"/>
       </xacro:if>
       <dynamics damping="0.0" friction="0.0"/>
@@ -207,5 +207,5 @@
       </xacro:unless>
       <xacro:if value="${joint_limited}">
-        <limit lower="${0}" upper="${pi}" effort="54.0" velocity="3.2"/>
+        <limit lower="${-110.0*pi/180.0}" upper="${0}" effort="54.0" velocity="3.2"/>
       </xacro:if>
       <dynamics damping="0.0" friction="0.0"/>

Commit message: Putting initial rail position on the other side of the table

File: excel_description/urdf/table_rail.urdf.xacro (robot description, xacro)
@@ -14,6 +14,7 @@
    <!-- Kinematic model -->
    <property name="rail_length" value="3.54" />
-   <!-- Collision model -->
-   <property name="table_collision_offset" value="0.135 0.81 0.935" />
+   <!-- Collision model
+   <property name="table_collision_offset" value="0.135 0.81 0.935" />-->
+   <property name="table_collision_offset" value="3.675 0.81 0.935" />
    <xacro:macro name="table_rail" params="prefix">
       <link name="${prefix}table_link">
@@ -34,5 +35,5 @@
          <parent link="${prefix}table_link" />
          <child link="${prefix}rail_link" />
-         <origin rpy="0.0 0.0 0.0" xyz="${table_collision_offset}" />
+         <origin rpy="0.0 0.0 ${pi}" xyz="${table_collision_offset}" />
          <axis xyz="1 0 0" />
          <limit effort="10.0" lower="0.0" upper="${rail_length}" velocity="${pi}" />
@@ -48,5 +49,5 @@
          <parent link="${prefix}rail_link" />
          <child link="${prefix}base_link" />
-         <origin rpy="0.0 0.0 0.0" xyz="0.0 0.0 0.0" />
+         <origin rpy="0.0 0.0 ${pi}" xyz="0.0 0.0 0.0" />
       </joint>
       <xacro:table_rail_transmission prefix="${prefix}" />

Commit message: Fixing table_rail model offsets
Didn't account for rail plates/carriage.  Also rail needed shifting down axis by 55mm.

File: excel_description/urdf/table_rail.urdf.xacro (robot description, xacro)
@@ -17,5 +17,5 @@
    <!-- Collision model
    <property name="table_collision_offset" value="0.135 0.81 0.935" />-->
-   <property name="table_collision_offset" value="3.675 0.81 0.935" />
+   <property name="table_collision_offset" value="3.620 0.81 0.935" />
    <xacro:macro name="table_rail" params="prefix">
       <link name="${prefix}table_link">
@@ -50,5 +50,5 @@
          <parent link="${prefix}rail_link" />
          <child link="${prefix}base_link" />
-         <origin rpy="0.0 0.0 ${pi}" xyz="0.0 0.0 0.0" />
+         <origin rpy="0.0 0.0 ${pi}" xyz="0.0 0.0 0.034" />
       </joint>
       <xacro:table_rail_transmission prefix="${prefix}" />

Commit message: Fixing table_rail include bugs for xacro files.

File: excel_description/urdf/table_rail.urdf.xacro (robot description, xacro)
@@ -5,7 +5,4 @@
 -->
 <robot xmlns:xacro="http://ros.org/wiki/xacro">
-   <xacro:include filename="$(find excel_description)/urdf/table_rail.transmission.xacro" />
-   <xacro:include filename="$(find excel_description)/urdf/table_rail.gazebo.xacro" />
-   <!--<xacro:include filename="$(find ur_description)/urdf/materials.urdf.xacro" />-->
    <property name="pi" value="3.14159265" />
    <property name="scale" value="0.001 0.001 0.001" />
@@ -18,5 +15,5 @@
    <property name="table_collision_offset" value="0.135 0.81 0.935" />-->
    <property name="table_collision_offset" value="3.620 0.81 0.935" />
-   <xacro:macro name="table_rail" params="prefix">
+   <xacro:macro name="table_rail">
       <link name="table_link">
          <visual>

Commit message: Adding the ceiling in the tables collision

File: excel_description/urdf/table_rail.urdf.xacro (robot description, xacro)
@@ -53,4 +53,10 @@
             <origin xyz="1.847 0.811 0.905" rpy="0 0 0" />
          </collision>
+         <collision>
+            <geometry>
+              <box size="4.0 2.0 0.2" />
+            </geometry>
+            <origin xyz="2.0 1.0 1.9" rpy="0 0 0" />
+         </collision>
       </link>
       <joint name="table_rail_joint" type="prismatic">
