Commit message: Fixing gripper joints and renaming excel_bringup

File: excel_description/urdf/gripper.urdf.xacro (robot description, xacro)
@@ -54,5 +54,5 @@
          </visual>
       </link>
-      <joint name="${prefix}robotiq_85_left_knuckle_joint" type="revolute">
+      <joint name="${prefix}robotiq_85_left_knuckle_joint" type="fixed">
          <parent link="${prefix}robotiq_85_base_link" />
          <child link="${prefix}robotiq_85_left_knuckle_link" />
@@ -74,5 +74,5 @@
          </visual>
       </link>
-      <joint name="${prefix}robotiq_85_right_knuckle_joint" type="revolute">
+      <joint name="${prefix}robotiq_85_right_knuckle_joint" type="fixed">
          <parent link="${prefix}robotiq_85_base_link" />
          <child link="${prefix}robotiq_85_right_knuckle_link" />
@@ -135,5 +135,5 @@
          </visual>
       </link>
-      <joint name="${prefix}robotiq_85_left_inner_knuckle_joint" type="revolute">
+      <joint name="${prefix}robotiq_85_left_inner_knuckle_joint" type="fixed">
          <parent link="${prefix}robotiq_85_base_link" />
          <child link="${prefix}robotiq_85_left_inner_knuckle_link" />
@@ -156,5 +156,5 @@
          </visual>
       </link>
-      <joint name="${prefix}robotiq_85_right_inner_knuckle_joint" type="revolute">
+      <joint name="${prefix}robotiq_85_right_inner_knuckle_joint" type="fixed">
          <parent link="${prefix}robotiq_85_base_link" />
          <child link="${prefix}robotiq_85_right_inner_knuckle_link" />
@@ -177,5 +177,5 @@
          </visual>
       </link>
-      <joint name="${prefix}robotiq_85_left_finger_tip_joint" type="revolute">
+      <joint name="${prefix}robotiq_85_left_finger_tip_joint" type="fixed">
          <parent link="${prefix}robotiq_85_left_inner_knuckle_link" />
          <child link="${prefix}robotiq_85_left_finger_tip_link" />
@@ -198,5 +198,5 @@
          </visual>
       </link>
-      <joint name="${prefix}robotiq_85_right_finger_tip_joint" type="revolute">
+      <joint name="${prefix}robotiq_85_right_finger_tip_joint" type="fixed">
          <parent link="${prefix}robotiq_85_right_inner_knuckle_link" />
          <child link="${prefix}robotiq_85_right_finger_tip_link" />

Commit message: Adding a gripper controller, and gripping actions in the main nodes

File: excel_description/urdf/gripper.urdf.xacro (robot description, xacro)
@@ -65,5 +65,5 @@
          </collision>
       </link>
-      <joint name="${prefix}robotiq_85_left_knuckle_joint" type="fixed">
+      <joint name="${prefix}robotiq_85_left_knuckle_joint" type="revolute">
          <parent link="${prefix}robotiq_85_base_link" />
          <child link="${prefix}robotiq_85_left_knuckle_link" />
@@ -85,5 +85,5 @@
          </visual>
       </link>
-      <joint name="${prefix}robotiq_85_right_knuckle_joint" type="fixed">
+      <joint name="${prefix}robotiq_85_right_knuckle_joint" type="revolute">
          <parent link="${prefix}robotiq_85_base_link" />
          <child link="${prefix}robotiq_85_right_knuckle_link" />
@@ -106,5 +106,5 @@
          </visual>
       </link>
-      <joint name="${prefix}robotiq_85_left_finger_joint" type="fixed">
+      <joint name="${prefix}robotiq_85_left_finger_joint" type="revolute">
          <parent link="${prefix}robotiq_85_left_knuckle_link" />
          <child link="${prefix}robotiq_85_left_finger_link" />
@@ -126,5 +126,5 @@
          </visual>
       </link>
-      <joint name="${prefix}robotiq_85_right_finger_joint" type="fixed">
+      <joint name="${prefix}robotiq_85_right_finger_joint" type="revolute">
          <parent link="${prefix}robotiq_85_right_knuckle_link" />
          <child link="${prefix}robotiq_85_right_finger_link" />
@@ -146,5 +146,5 @@
          </visual>
       </link>
-      <joint name="${prefix}robotiq_85_left_inner_knuckle_joint" type="fixed">
+      <joint name="${prefix}robotiq_85_left_inner_knuckle_joint" type="revolute">
          <parent link="${prefix}robotiq_85_base_link" />
          <child link="${prefix}robotiq_85_left_inner_knuckle_link" />
@@ -167,5 +167,5 @@
          </visual>
       </link>
-      <joint name="${prefix}robotiq_85_right_inner_knuckle_joint" type="fixed">
+      <joint name="${prefix}robotiq_85_right_inner_knuckle_joint" type="revolute">
          <parent link="${prefix}robotiq_85_base_link" />
          <child link="${prefix}robotiq_85_right_inner_knuckle_link" />
@@ -188,5 +188,5 @@
          </visual>
       </link>
-      <joint name="${prefix}robotiq_85_left_finger_tip_joint" type="fixed">
+      <joint name="${prefix}robotiq_85_left_finger_tip_joint" type="revolute">
          <parent link="${prefix}robotiq_85_left_inner_knuckle_link" />
          <child link="${prefix}robotiq_85_left_finger_tip_link" />
@@ -215,5 +215,5 @@
          </collision>
       </link>
-      <joint name="${prefix}robotiq_85_right_finger_tip_joint" type="fixed">
+      <joint name="${prefix}robotiq_85_right_finger_tip_joint" type="revolute">
          <parent link="${prefix}robotiq_85_right_inner_knuckle_link" />
          <child link="${prefix}robotiq_85_right_finger_tip_link" />

Commit message: Switching gripper joints from revolute to fixed

File: excel_description/urdf/gripper.urdf.xacro (robot description, xacro)
@@ -65,5 +65,5 @@
          </collision>
       </link>
-      <joint name="${prefix}robotiq_85_left_knuckle_joint" type="revolute">
+      <joint name="${prefix}robotiq_85_left_knuckle_joint" type="fixed">
          <parent link="${prefix}robotiq_85_base_link" />
          <child link="${prefix}robotiq_85_left_knuckle_link" />
@@ -85,5 +85,5 @@
          </visual>
       </link>
-      <joint name="${prefix}robotiq_85_right_knuckle_joint" type="revolute">
+      <joint name="${prefix}robotiq_85_right_knuckle_joint" type="fixed">
          <parent link="${prefix}robotiq_85_base_link" />
          <child link="${prefix}robotiq_85_right_knuckle_link" />
@@ -106,5 +106,5 @@
          </visual>
       </link>
-      <joint name="${prefix}robotiq_85_left_finger_joint" type="revolute">
+      <joint name="${prefix}robotiq_85_left_finger_joint" type="fixed">
          <parent link="${prefix}robotiq_85_left_knuckle_link" />
          <child link="${prefix}robotiq_85_left_finger_link" />
@@ -126,5 +126,5 @@
          </visual>
       </link>
-      <joint name="${prefix}robotiq_85_right_finger_joint" type="revolute">
+      <joint name="${prefix}robotiq_85_right_finger_joint" type="fixed">
          <parent link="${prefix}robotiq_85_right_knuckle_link" />
          <child link="${prefix}robotiq_85_right_finger_link" />
@@ -146,5 +146,5 @@
          </visual>
       </link>
-      <joint name="${prefix}robotiq_85_left_inner_knuckle_joint" type="revolute">
+      <joint name="${prefix}robotiq_85_left_inner_knuckle_joint" type="fixed">
          <parent link="${prefix}robotiq_85_base_link" />
          <child link="${prefix}robotiq_85_left_inner_knuckle_link" />
@@ -167,5 +167,5 @@
          </visual>
       </link>
-      <joint name="${prefix}robotiq_85_right_inner_knuckle_joint" type="revolute">
+      <joint name="${prefix}robotiq_85_right_inner_knuckle_joint" type="fixed">
          <parent link="${prefix}robotiq_85_base_link" />
          <child link="${prefix}robotiq_85_right_inner_knuckle_link" />
@@ -188,5 +188,5 @@
          </visual>
       </link>
-      <joint name="${prefix}robotiq_85_left_finger_tip_joint" type="revolute">
+      <joint name="${prefix}robotiq_85_left_finger_tip_joint" type="fixed">
          <parent link="${prefix}robotiq_85_left_inner_knuckle_link" />
          <child link="${prefix}robotiq_85_left_finger_tip_link" />
@@ -215,5 +215,5 @@
          </collision>
       </link>
-      <joint name="${prefix}robotiq_85_right_finger_tip_joint" type="revolute">
+      <joint name="${prefix}robotiq_85_right_finger_tip_joint" type="fixed">
          <parent link="${prefix}robotiq_85_right_inner_knuckle_link" />
          <child link="${prefix}robotiq_85_right_finger_tip_link" />

Commit message: Reducing the gripper collision model

File: excel_description/urdf/gripper.urdf.xacro (robot description, xacro)
@@ -210,5 +210,5 @@
          <collision>
             <geometry>
-              <box size="0.038 0.12 0.05" />
+              <box size="0.038 0.12 0.035" />
             </geometry>
             <origin xyz="0.01 0.00 0" rpy="0 0 0" />
@@ -237,5 +237,5 @@
          <collision>
             <geometry>
-              <box size="0.038 0.12 0.05" />
+              <box size="0.038 0.12 0.035" />
             </geometry>
             <origin xyz="-0.01 0.00 0" rpy="0 0 0" />
