Commit message: Adding the real calibration frame position values to the urdf

File: excel_description/urdf/cameras.urdf.xacro (robot description, xacro)
@@ -12,5 +12,5 @@
          <parent link="${prefix}table_link" />
          <child link="${prefix}45_camera_link" />
-         <origin rpy="${pi} 0.0 0.0" xyz="0.53 1.42 2.52" />
+         <origin rpy="3.1358844265653847 -0.04203340790110574 -0.013879785230443352" xyz="0.569 1.521 2.597" />
       </joint>
       <link name="${prefix}35_camera_link">
@@ -19,19 +19,19 @@
          <parent link="${prefix}table_link" />
          <child link="${prefix}35_camera_link" />
-         <origin rpy="${pi} 0.0 0.0" xyz="1.59 0.11 2.63" />
+         <origin rpy="3.107697904738654 -0.03808611429915326 -0.005354382539543283" xyz="1.625 0.149 2.643" />
       </joint>
-      <link name="${prefix}kinect_1_link">
+      <link name="${prefix}kinect_front_link">
       </link>
-      <joint name="${prefix}kinect_1_joint" type="fixed">
+      <joint name="${prefix}kinect_front_joint" type="fixed">
          <parent link="${prefix}table_link" />
-         <child link="${prefix}kinect_1_link" />
-         <origin rpy="0.0 0.0 0.0" xyz="3 3 3" />
+         <child link="${prefix}kinect_front_link" />
+         <origin rpy="-2.0911526920812413 0.018717144155139063 -1.4733313495598332" xyz="-1.096 1.559 2.344" />
       </joint>
-      <link name="${prefix}kinect_2_link">
+      <link name="${prefix}kinect_back_link">
       </link>
-      <joint name="${prefix}kinect_2_joint" type="fixed">
+      <joint name="${prefix}kinect_back_joint" type="fixed">
          <parent link="${prefix}table_link" />
-         <child link="${prefix}kinect_2_link" />
-         <origin rpy="0.0 0.0 0.0" xyz="2 2 2" />
+         <child link="${prefix}kinect_back_link" />
+         <origin rpy="-2.1746265277559695 0.01568256219680734 2.0515498028502073" xyz="3.848 3.690 2.314" />
       </joint>
       <link name="${prefix}gripper_camera_link">

Commit message: Cleaning up URDF files. Fixing camera calibrations.

File: excel_description/urdf/cameras.urdf.xacro (robot description, xacro)
@@ -1,43 +1,42 @@
 <?xml version="1.0" encoding="UTF-8"?>
 <!--
-  Author: Jimmy Da Silva
-  Contributers: Kelsey Hawkins, Ajit Krisshna N L, Muhammad Asif Rana
+  Authors: Jimmy Da Silva, Kelsey Hawkins
 -->
 <robot xmlns:xacro="http://ros.org/wiki/xacro">
    <property name="pi" value="3.14159265" />
-   <xacro:macro name="cameras" params="prefix">
-      <link name="${prefix}45_camera_link">
+   <xacro:macro name="cameras">
+      <link name="overhead_hum_ws_frame">
       </link>
-      <joint name="${prefix}45_camera_joint" type="fixed">
-         <parent link="${prefix}table_link" />
-         <child link="${prefix}45_camera_link" />
-         <origin rpy="3.1358844265653847 -0.04203340790110574 -0.013879785230443352" xyz="0.569 1.521 2.597" />
+      <joint name="overhead_hum_ws_cam_joint" type="fixed">
+         <parent link="table_link" />
+         <child link="overhead_hum_ws_frame" />
+         <origin rpy="3.136 -0.042 -0.014" xyz="0.569 1.521 2.597" />
       </joint>
-      <link name="${prefix}35_camera_link">
+      <link name="overhead_rob_ws_frame">
       </link>
-      <joint name="${prefix}35_camera_joint" type="fixed">
-         <parent link="${prefix}table_link" />
-         <child link="${prefix}35_camera_link" />
-         <origin rpy="3.107697904738654 -0.03808611429915326 -0.005354382539543283" xyz="1.625 0.149 2.643" />
+      <joint name="overhead_rob_ws_cam_joint" type="fixed">
+         <parent link="table_link" />
+         <child link="overhead_rob_ws_frame" />
+         <origin rpy="3.108 -0.038 -0.005" xyz="1.625 0.149 2.643" />
       </joint>
-      <link name="${prefix}kinect_front_link">
+      <link name="kinect_front_link">
       </link>
-      <joint name="${prefix}kinect_front_joint" type="fixed">
-         <parent link="${prefix}table_link" />
-         <child link="${prefix}kinect_front_link" />
-         <origin rpy="-2.0911526920812413 0.018717144155139063 -1.4733313495598332" xyz="-1.096 1.559 2.344" />
+      <joint name="kinect_front_joint" type="fixed">
+         <parent link="table_link" />
+         <child link="kinect_front_link" />
+         <origin rpy="0.022 0.520 0.108" xyz="-1.100 1.604 2.345" />
       </joint>
-      <link name="${prefix}kinect_back_link">
+      <link name="kinect_back_link">
       </link>
-      <joint name="${prefix}kinect_back_joint" type="fixed">
-         <parent link="${prefix}table_link" />
-         <child link="${prefix}kinect_back_link" />
-         <origin rpy="-2.1746265277559695 0.01568256219680734 2.0515498028502073" xyz="3.848 3.690 2.314" />
+      <joint name="kinect_back_joint" type="fixed">
+         <parent link="table_link" />
+         <child link="kinect_back_link" />
+         <origin rpy="0.019 0.604 -2.650" xyz="3.869 3.650 2.315" />
       </joint>
-      <link name="${prefix}gripper_camera_link">
+      <link name="gripper_camera_link">
       </link>
-      <joint name="${prefix}gripper_camera_joint" type="fixed">
-         <parent link="${prefix}ee_link" />
-         <child link="${prefix}gripper_camera_link" />
+      <joint name="gripper_camera_joint" type="fixed">
+         <parent link="ee_link" />
+         <child link="gripper_camera_link" />
          <origin rpy="0.0 0.0 0.0" xyz="0.1 0.1 0.1" />
       </joint>

File: excel_description/urdf/excel_robot.urdf.xacro (robot description, xacro)
@@ -25,8 +25,8 @@
   />
    <!-- table&rail -->
-   <xacro:table_rail prefix="" />
+   <xacro:table_rail/>
    <!-- gripper -->
    <xacro:gripper prefix="" />
    <!-- cameras -->
-   <xacro:cameras prefix="" />
+   <xacro:cameras/>
 </robot>

File: excel_description/urdf/excel_robot_moplan.urdf.xacro (robot description, xacro)
@@ -25,8 +25,8 @@
   />
    <!-- table&rail -->
-   <xacro:table_rail prefix="" />
+   <xacro:table_rail/>
    <!-- gripper -->
    <xacro:gripper prefix="" />
    <!-- cameras -->
-   <xacro:cameras prefix="" />
+   <xacro:cameras/>
 </robot>

File: excel_description/urdf/gripper.urdf.xacro (robot description, xacro)
@@ -1,6 +1,5 @@
 <?xml version="1.0" encoding="UTF-8"?>
 <!--
-  Author: Jimmy Da Silva
-  Contributers: Kelsey Hawkins, Ajit Krisshna N L, Muhammad Asif Rana
+  Courtesy of JHU: https://github.com/jhu-lcsr/robotiq
 -->
 <robot xmlns:xacro="http://ros.org/wiki/xacro">

File: excel_description/urdf/table_rail.urdf.xacro (robot description, xacro)
@@ -19,5 +19,5 @@
    <property name="table_collision_offset" value="3.620 0.81 0.935" />
    <xacro:macro name="table_rail" params="prefix">
-      <link name="${prefix}table_link">
+      <link name="table_link">
          <visual>
             <geometry>
@@ -33,7 +33,7 @@
          </collision>
       </link>
-      <joint name="${prefix}table_rail_joint" type="prismatic">
-         <parent link="${prefix}table_link" />
-         <child link="${prefix}rail_link" />
+      <joint name="table_rail_joint" type="prismatic">
+         <parent link="table_link" />
+         <child link="rail_link" />
          <origin rpy="0.0 0.0 ${pi}" xyz="${table_collision_offset}" />
          <axis xyz="1 0 0" />
@@ -41,5 +41,5 @@
          <dynamics damping="10" friction="0.1" />
       </joint>
-      <link name="${prefix}rail_link">
+      <link name="rail_link">
          <inertial>
             <mass value="${rail_mass}" />
@@ -47,11 +47,18 @@
          </inertial>
       </link>
-      <joint name="${prefix}rail_base_joint" type="fixed">
-         <parent link="${prefix}rail_link" />
-         <child link="${prefix}base_link" />
+      <joint name="rail_base_joint" type="fixed">
+         <parent link="rail_link" />
+         <child link="base_link" />
          <origin rpy="0.0 0.0 ${pi}" xyz="0.0 0.0 0.034" />
       </joint>
-      <xacro:table_rail_transmission prefix="${prefix}" />
-      <xacro:table_rail_gazebo prefix="${prefix}" />
+      <transmission name="rail_base_trans" type="pr2_mechanism_model/SimpleTransmission">
+         <actuator name="rail_base_motor" />
+         <joint name="rail_base_joint" />
+         <mechanicalReduction>1</mechanicalReduction>
+      </transmission>
+      <gazebo reference="table_link">
+         <material value="Gazebo/Blue " />
+         <turnGravityOff>false</turnGravityOff>
+      </gazebo>
    </xacro:macro>
 </robot>

Commit message: Fixing camera focal plan position

File: excel_description/urdf/cameras.urdf.xacro (robot description, xacro)
@@ -42,5 +42,12 @@
          <parent link="ee_link" />
          <child link="gripper_camera_link" />
-         <origin rpy="0.0 0.0 0.0" xyz="0.1 0.1 0.1" />
+         <origin rpy="0.0 0.0 0.0" xyz="0.015 -0.02 0.06" />
+      </joint>
+      <link name="gripper_camera_focal_link">
+      </link>
+      <joint name="gripper_camera_focal_joint" type="fixed">
+         <parent link="gripper_camera_link" />
+         <child link="gripper_camera_focal_link" />
+         <origin rpy="0.0 0.0 0.0" xyz="0.0 1.0 0.0" />
       </joint>
    </xacro:macro>

Commit message: Updating overhead_rob extrinsics

File: excel_description/urdf/cameras.urdf.xacro (robot description, xacro)
@@ -19,5 +19,6 @@
          <parent link="table_link" />
          <child link="overhead_rob_ws_frame" />
-         <origin rpy="3.108 -0.038 -0.005" xyz="1.625 0.149 2.643" />
+         <!--<origin rpy="3.108 -0.038 -0.005" xyz="1.625 0.149 2.643" />-->
+         <origin rpy="3.108 -0.028 -0.025" xyz="1.624 0.12 2.643" />
       </joint>
       <link name="kinect_front_link">

Commit message: Adding args to shift quickly the cameras positions

File: excel_description/urdf/cameras.urdf.xacro (robot description, xacro)
@@ -6,5 +6,5 @@
    <xacro:include filename="$(find excel_description)/urdf/kinect_frames.urdf.xacro" />
    <property name="pi" value="3.14159265" />
-   <xacro:macro name="cameras">
+   <xacro:macro name="cameras" params="x_offset y_offset theta_offset">
       <link name="overhead_hum_ws_frame">
       </link>
@@ -12,5 +12,5 @@
          <parent link="table_link" />
          <child link="overhead_hum_ws_frame" />
-         <origin rpy="3.136 -0.042 -0.014" xyz="0.569 1.521 2.597" />
+         <origin rpy="3.136 -0.042 ${-0.014+theta_offset}" xyz="${0.569+x_offset} ${1.521+y_offset} 2.597" />
       </joint>
       <link name="overhead_rob_ws_frame">
@@ -20,5 +20,5 @@
          <child link="overhead_rob_ws_frame" />
          <!--<origin rpy="3.108 -0.038 -0.005" xyz="1.625 0.149 2.643" />-->
-         <origin rpy="3.108 -0.028 -0.025" xyz="1.624 0.12 2.643" />
+         <origin rpy="3.108 -0.028 ${-0.025+theta_offset}" xyz="${1.624+x_offset} ${0.12+y_offset} 2.643" />
       </joint>
       <link name="kinect_front_link">

File: excel_description/urdf/excel_robot_moplan.urdf.xacro (robot description, xacro)
@@ -29,4 +29,4 @@
    <xacro:gripper prefix="" />
    <!-- cameras -->
-   <xacro:cameras/>
+   <xacro:cameras x_offset="0.0" y_offset="0.0" theta_offset="0.0"/>
 </robot>

Commit message: Publishing again gripper_camera_focal_link

File: excel_description/urdf/cameras.urdf.xacro (robot description, xacro)
@@ -7,4 +7,5 @@
    <property name="pi" value="3.14159265" />
    <xacro:macro name="cameras" params="x_offset y_offset theta_offset">
+<!--
       <link name="overhead_hum_ws_frame">
       </link>
@@ -19,5 +20,4 @@
          <parent link="table_link" />
          <child link="overhead_rob_ws_frame" />
-         <!--<origin rpy="3.108 -0.038 -0.005" xyz="1.625 0.149 2.643" />-->
          <origin rpy="3.108 -0.028 ${-0.025+theta_offset}" xyz="${1.624+x_offset} ${0.12+y_offset} 2.643" />
       </joint>
@@ -38,4 +38,5 @@
       </joint>
       <xacro:kinect_frames camera="kinect_back"/>
+-->
       <link name="gripper_camera_link">
       </link>

File: excel_description/urdf/excel_robot_moplan.urdf.xacro (robot description, xacro)
@@ -14,5 +14,5 @@
    <xacro:include filename="$(find excel_description)/urdf/gripper.urdf.xacro" />
    <!-- include cameras -->
-   <!-- <xacro:include filename="$(find excel_description)/urdf/cameras.urdf.xacro" /> -->
+   <xacro:include filename="$(find excel_description)/urdf/cameras.urdf.xacro" />
    <!-- ur10 -->
   <xacro:ur10_robot prefix="" cylinders_collision="true"
@@ -29,4 +29,4 @@
    <xacro:gripper prefix="" />
    <!-- cameras -->
-   <!-- <xacro:cameras x_offset="0.0" y_offset="0.0" theta_offset="0.0"/> -->
+   <xacro:cameras x_offset="0.0" y_offset="0.0" theta_offset="0.0"/>
 </robot>
